Commit message: success to 0.1m/s walking

File: dyros_tocabi_v2/tocabi_description/robots/dyros_tocabi.urdf (robot description, URDF)
Before this commit: robot dyros_tocabi_description, 36 links, 35 joints
Joints:
- joint Head_Joint: limit lower=-1.54 upper=1.54 effort=500 velocity=100 -> lower=-1.54 upper=1.54 effort=500 velocity=3.14
- joint L_AnklePitch_Joint: limit lower=-3.14 upper=3.14 effort=500 velocity=100 -> lower=-1.57 upper=1.57 effort=500 velocity=3.14
- joint L_AnkleRoll_Joint: limit lower=-3.14 upper=3.14 effort=500 velocity=100 -> lower=-1.57 upper=1.57 effort=500 velocity=3.14
- joint L_Armlink_Joint: limit lower=-3.14159 upper=3.14159 effort=500 velocity=100 -> lower=-3.14159 upper=3.14159 effort=500 velocity=3.14
- joint L_Elbow_Joint: limit lower=-3.14159 upper=2.8 effort=500 velocity=100 -> lower=-3.14159 upper=2.8 effort=500 velocity=3.14
- joint L_Foot_Joint: limit lower=-3.14 upper=3.14 effort=500 velocity=100 -> lower=-1.57 upper=1.57 effort=500 velocity=3.14
- joint L_Forearm_Joint: limit lower=-3.14159 upper=3.14159 effort=500 velocity=100 -> lower=-3.14159 upper=3.14159 effort=500 velocity=3.14
- joint L_HipPitch_Joint: limit lower=-3.14 upper=3.14 effort=500 velocity=100 -> lower=-1.57 upper=1.57 effort=500 velocity=3.14
- joint L_HipRoll_Joint: limit lower=-3.14 upper=3.14 effort=500 velocity=100 -> lower=-1.57 upper=1.57 effort=500 velocity=3.14
- joint L_HipYaw_Joint: limit lower=-3.14 upper=3.14 effort=500 velocity=100 -> lower=-1.57 upper=1.57 effort=500 velocity=3.14
- joint L_Knee_Joint: limit lower=-3.14 upper=3.14 effort=500 velocity=100 -> lower=0.0 upper=1.57 effort=500 velocity=3.14
- joint L_Shoulder1_Joint: limit lower=-2.09 upper=1.54 effort=500 velocity=100 -> lower=-2.09 upper=1.54 effort=500 velocity=3.14
- joint L_Shoulder2_Joint: limit lower=-3.14159 upper=3.14159 effort=500 velocity=100 -> lower=-3.14159 upper=3.14159 effort=500 velocity=3.14
- joint L_Shoulder3_Joint: limit lower=-1.9199 upper=1.9199 effort=500 velocity=100 -> lower=-1.9199 upper=1.9199 effort=500 velocity=3.14
- joint L_Wrist1_Joint: limit lower=-3.14159 upper=3.14159 effort=500 velocity=100 -> lower=-3.14159 upper=3.14159 effort=500 velocity=3.14
- joint L_Wrist2_Joint: limit lower=-2.094 upper=2.094 effort=500 velocity=100 -> lower=-2.094 upper=2.094 effort=500 velocity=3.14
- joint Neck_Joint: limit lower=-1.54 upper=1.54 effort=500 velocity=100 -> lower=-1.54 upper=1.54 effort=500 velocity=3.14
- joint R_AnklePitch_Joint: limit lower=-3.14 upper=3.14 effort=500 velocity=100 -> lower=-1.57 upper=1.57 effort=500 velocity=3.14
- joint R_AnkleRoll_Joint: limit lower=-3.14 upper=3.14 effort=500 velocity=100 -> lower=-1.57 upper=1.57 effort=500 velocity=3.14
- joint R_Armlink_Joint: limit lower=-3.14159 upper=3.14159 effort=500 velocity=100 -> lower=-3.14159 upper=3.14159 effort=500 velocity=3.14
- joint R_Elbow_Joint: limit lower=-2.967 upper=3.14159 effort=500 velocity=100 -> lower=-2.967 upper=3.14159 effort=500 velocity=3.14
- joint R_Foot_Joint: limit lower=-3.14 upper=3.14 effort=500 velocity=100 -> lower=-1.57 upper=1.57 effort=500 velocity=3.14
- joint R_Forearm_Joint: limit lower=-3.14159 upper=3.14159 effort=500 velocity=100 -> lower=-3.14159 upper=3.14159 effort=500 velocity=3.14
- joint R_HipPitch_Joint: limit lower=-3.14 upper=3.14 effort=500 velocity=100 -> lower=-1.57 upper=1.57 effort=500 velocity=3.14
- joint R_HipRoll_Joint: limit lower=-3.14 upper=3.14 effort=500 velocity=100 -> lower=-1.57 upper=1.57 effort=500 velocity=3.14
- joint R_HipYaw_Joint: limit lower=-3.14 upper=3.14 effort=500 velocity=100 -> lower=-1.57 upper=1.57 effort=500 velocity=3.14
- joint R_Knee_Joint: limit lower=-3.14 upper=3.14 effort=500 velocity=100 -> lower=0.0 upper=1.57 effort=500 velocity=3.14
- joint R_Shoulder1_Joint: limit lower=-1.54 upper=2.09 effort=500 velocity=100 -> lower=-1.54 upper=2.09 effort=500 velocity=3.14
- joint R_Shoulder2_Joint: limit lower=-3.14159 upper=3.14159 effort=500 velocity=100 -> lower=-3.14159 upper=3.14159 effort=500 velocity=3.14
- joint R_Shoulder3_Joint: limit lower=-1.9199 upper=1.9199 effort=500 velocity=100 -> lower=-1.9199 upper=1.9199 effort=500 velocity=3.14
- joint R_Wrist1_Joint: limit lower=-3.14159 upper=3.14159 effort=500 velocity=100 -> lower=-3.14159 upper=3.14159 effort=500 velocity=3.14
- joint R_Wrist2_Joint: limit lower=-2.094 upper=2.094 effort=500 velocity=100 -> lower=-2.094 upper=2.094 effort=500 velocity=3.14
- joint Upperbody_Joint: limit lower=-2.094 upper=2.094 effort=500 velocity=100 -> lower=-2.094 upper=2.094 effort=500 velocity=3.14
- joint Waist1_Joint: limit lower=-2.094 upper=2.094 effort=500 velocity=100 -> lower=-2.094 upper=2.094 effort=500 velocity=3.14
- joint Waist2_Joint: limit lower=-2.094 upper=2.094 effort=500 velocity=100 -> lower=-2.094 upper=2.094 effort=500 velocity=3.14

Commit message: [IJCAS] - hand/foot trajectory experiments

File: dyros_tocabi_v2/tocabi_description/robots/dyros_tocabi.urdf (robot description, URDF)
Before this commit: robot dyros_tocabi_description, 36 links, 35 joints
Links:
- link Head_Link: geometry collision cylinder length=0.043 radius=0.07
- link L_AnkleCenter_Link: geometry collision box size=0.1045 0.06 0.095; visual mesh filename=../meshes/AnkleCenter_L_Link.STL
- link L_AnkleRoll_Link: geometry collision cylinder length=0.0625 radius=0.045; visual mesh filename=../meshes/AnkleRoll_L_Link.STL
- link L_Armlink_Link: geometry collision cylinder length=0.16 radius=0.04; visual mesh filename=../meshes/L_arm.STL
- link L_Elbow_Link: geometry collision cylinder length=0.08 radius=0.04; collision cylinder length=0.08 radius=0.04
- link L_Foot_Link: geometry collision box size=0.3 0.17 0.027; collision cylinder length=0.0625 radius=0.045
- link L_Forearm_Link: geometry collision cylinder length=0.08 radius=0.025; collision cylinder length=0.1 radius=0.04
- link L_HipCenter_Link: geometry collision box size=0.1045 0.06 0.095; visual mesh filename=../meshes/HipCenter_L_Link.STL
- link L_HipRoll_Link: geometry collision box size=0.012 0.072 0.095; collision box size=0.012 0.072 0.095
- link L_Knee_Link: geometry collision cylinder length=0.200 radius=0.06; visual mesh filename=../meshes/Knee_L_Link.STL
- link L_Shoulder1_Link: geometry collision cylinder length=0.11 radius=0.04; visual mesh filename=../meshes/L_shoulder1.STL
- link L_Shoulder2_Link: geometry collision cylinder length=0.05 radius=0.04; visual mesh filename=../meshes/L_shoulder2.STL
- link L_Shoulder3_Link: geometry collision cylinder length=0.12 radius=0.04; visual mesh filename=../meshes/L_shoulder3.STL
- link L_Thigh_Link: geometry collision cylinder length=0.07763 radius=0.049; collision cylinder length=0.2175 radius=0.06
- link L_Wrist1_Link: geometry collision cylinder length=0.06 radius=0.02; visual mesh filename=../meshes/L_wrist1.STL
- link Neck_Link: geometry collision cylinder length=0.043 radius=0.07; visual mesh filename=../meshes/neck.STL
- link Pelvis_Link: geometry collision box size=0.141 0.305 0.05; collision cylinder length=0.088 radius=0.045
- link R_AnkleCenter_Link: geometry collision box size=0.1045 0.06 0.095; visual mesh filename=../meshes/AnkleCenter_R_Link.STL
- link R_AnkleRoll_Link: geometry collision cylinder length=0.0625 radius=0.045; visual mesh filename=../meshes/AnkleRoll_R_Link.STL
- link R_Armlink_Link: geometry collision cylinder length=0.16 radius=0.04; visual mesh filename=../meshes/R_arm.STL
- link R_Elbow_Link: geometry collision cylinder length=0.08 radius=0.04; collision cylinder length=0.08 radius=0.04
- link R_Foot_Link: geometry collision box size=0.3 0.17 0.027; collision cylinder length=0.0625 radius=0.045
- link R_Forearm_Link: geometry collision cylinder length=0.08 radius=0.025; collision cylinder length=0.1 radius=0.04
- link R_HipCenter_Link: geometry collision box size=0.1045 0.06 0.095; visual mesh filename=../meshes/HipCenter_R_Link.STL
- link R_HipRoll_Link: geometry collision box size=0.012 0.072 0.095; collision box size=0.012 0.072 0.095
- link R_Knee_Link: geometry collision cylinder length=0.200 radius=0.06; visual mesh filename=../meshes/Knee_R_Link.STL
- link R_Shoulder1_Link: geometry collision cylinder length=0.11 radius=0.04; visual mesh filename=../meshes/R_shoulder1.STL
- link R_Shoulder2_Link: geometry collision cylinder length=0.05 radius=0.04; visual mesh filename=../meshes/R_shoulder2.STL
- link R_Shoulder3_Link: geometry collision cylinder length=0.12 radius=0.04; visual mesh filename=../meshes/R_shoulder3.STL
- link R_Thigh_Link: geometry collision cylinder length=0.07763 radius=0.049; collision cylinder length=0.2175 radius=0.06
- link R_Wrist1_Link: geometry collision cylinder length=0.06 radius=0.02; visual mesh filename=../meshes/R_wrist1.STL
- link Upperbody_Link: geometry collision box size=0.12 0.07 0.14; collision box size=0.21 0.11 0.07
- link Waist1_Link: geometry collision box size=0.094 0.01 0.091; collision box size=0.094 0.01 0.091
- link Waist2_Link: geometry collision box size=0.09 0.1 0.091; collision box size=0.1 0.1 0.06
